File: charge-tester.kicad_pcb (KiCad board)
At the start: 2 copper layers, 85 x 56 mm, 76 parts, among them J1 Conn_01x02, J2 Conn_01x02, J3 Conn_01x02, J4 Conn_01x02, J5 Conn_01x06, Q1 IRFB4020, Q2 FDV303N, Q3 FDV303N, SW1 SW_Push, U1 TPS7B88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

Commit message: schematic: Switch op-amp to LM358BA
Parts:
- U3: value OPA1678 -> LM358
Changed lines of the file:
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@@
 			)
 		)
-		(property "Value" "OPA1678"
+		(property "Value" "LM358"
 			(at 0 3.4 90)
 			(layer "F.Fab")
@@
 			)
 		)
-		(property "Datasheet" "http://www.ti.com/lit/ds/symlink/opa1678.pdf"
+		(property "Datasheet" "http://www.ti.com/lit/ds/symlink/lm2904-n.pdf"
 			(at 0 0 90)
 			(layer "F.Fab")
@@
 			)
 		)
-		(property "Description" "Low-Distortion Audio Operational Amplifiers, SOIC-8/VSSOP-8"
+		(property "Description" "Low-Power, Dual Operational Amplifiers, DIP-8/SOIC-8/TO-99-8"
 			(at 0 0 90)
 			(layer "F.Fab")
@@
 			)
 		)
-		(property "Dist" "LCSC"
+		(property "Dist" "Mouser"
 			(at 0 0 270)
 			(unlocked yes)
@@
 			)
 		)
-		(property "Dist #" "C192421"
+		(property "Dist #" "595-LM358BAIDR"
 			(at 0 0 270)
 			(unlocked yes)
@@
 			)
 		)
-		(property "Mfr #" "OPA1678IDR"
+		(property "Mfr #" "LM358BAIDR"
 			(at 0 0 270)
 			(unlocked yes)
