File: charge-tester.kicad_sch (KiCad schematic)
At the start: 60 parts, among them J1 Conn_01x02, J2 Conn_01x02, J3 Conn_01x02, J4 Conn_01x02, J5 Conn_01x06, Q1 IRFB4020, Q2 FDV303N, Q3 FDV303N, U1 TPS7B88, U2 MCP1700x-330xxMB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

Commit message: schematic: Assign footprints and fill out BOM
Parts:
- removed Q2, Q3: FDV303N, symbol Simulation_SPICE:NMOS
- added Q2, Q3: FDV303N, Package_TO_SOT_SMD:SOT-23, symbol yfs:FDV303N
- C10, C9: footprint (none) -> Capacitor_SMD:C_0603_1608Metric; Dist (none) -> LCSC; Dist # (none) -> C85973; Mfr (none) -> Murata; Mfr # (none) -> GRM1885C1H103JA01D
- C7: footprint (none) -> Capacitor_SMD:C_0603_1608Metric; Dist (none) -> LCSC; Dist # (none) -> C5199872; Mfr (none) -> Samsung; Mfr # (none) -> CL10B105KB8NQNC
- C8: footprint (none) -> Capacitor_SMD:C_0603_1608Metric
- F1: Dist (none) -> LCSC; Dist # (none) -> C207019; Mfr (none) -> Littelfuse; Mfr # (none) -> 0805L010/24YR
- J3, J4: Dist # 538-215760-1022 -> 538-215760-1002; Mfr # 2157601022 -> 2157601002
- Q1: footprint (none) -> Package_TO_SOT_THT:TO-220-3_Vertical; Dist (none) -> LCSC; Dist # (none) -> C2649; Mfr (none) -> Infineon; Mfr # (none) -> IRFB4020PBF
- R10: footprint (none) -> Resistor_SMD:R_1206_3216Metric; Dist (none) -> LCSC; Dist # (none) -> C2903500; Mfr (none) -> Milliohm; Mfr # (none) -> HoJLR1206-1W-25mR-1%
- R11, R7, R8, R9: footprint (none) -> Resistor_SMD:R_0603_1608Metric; Dist (none) -> LCSC; Dist # (none) -> C21190; Mfr (none) -> Uni-Royal; Mfr # (none) -> 0603WAF1001T5E
- R12, R6: footprint (none) -> Resistor_SMD:R_0603_1608Metric; Dist (none) -> LCSC; Dist # (none) -> C25804; Mfr (none) -> Uni-Royal; Mfr # (none) -> 0603WAF1002T5E
- R2: footprint (none) -> Resistor_SMD:R_0603_1608Metric; Dist (none) -> LCSC; Dist # (none) -> C23138; Mfr (none) -> Uni-Royal; Mfr # (none) -> 0603WAF3300T5E
- R3, R4, R5: footprint (none) -> Resistor_SMD:R_0603_1608Metric
- RV1: footprint (none) -> Potentiometer_SMD:Potentiometer_Bourns_3269P_Horizontal
- U3: footprint (none) -> Package_SO:SOIC-8_3.9x4.9mm_P1.27mm; Dist (none) -> LCSC; Dist # (none) -> C192421; Mfr (none) -> Texas Instruments; Mfr # (none) -> OPA1678IDR
Connections:
- net GND: now also Q2.2 (S), Q3.2 (S)
- net at Q1.2 (G), R8.2: now also Q2.3 (D), Q3.3 (D)
- net at R11.1: now also Q3.1 (G)
- net at R7.2: now also Q2.1 (G)

Commit message: schematic: Add some more test points and net labels
Parts:
- added TP4, TP5, TP6, TP7, TP8: TestPoint, TestPoint:TestPoint_Keystone_5000-5004_Miniature, symbol Connector:TestPoint
Connections:
- net VBAT: now also TP7.1
- net VCC_SENSE: now also TP4.1
- net CC_FB: now reaches C10.2, R9.2, U3.6 (-)
- net CV_FB: now reaches C9.2, R3.2, R4.1, U3.2 (-)
- net at C8.1, R5.2, R6.1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: now also TP6.1
- net at C7.1, R2.2, U3.3 (+): now also TP5.1
- net GATE: now reaches Q1.2 (G), Q2.3 (D), Q3.3 (D), R8.2
- net GATE: now also TP8.1

Commit message: *: Initial layout
Parts:
- removed C15, C4: 1u, Capacitor_SMD:C_0603_1608Metric, symbol Device:C_Small
- removed Q1: IRFB4020, Package_TO_SOT_THT:TO-220-3_Vertical, symbol Simulation_SPICE:NMOS
- removed TP4: TestPoint, TestPoint:TestPoint_Keystone_5000-5004_Miniature, symbol Connector:TestPoint
- added C1: 100n, Capacitor_SMD:C_0603_1608Metric, symbol Device:C_Small
- added H1, H2, H3, H4: MountingHole_Pad, MountingHole:MountingHole_3.2mm_M3_Pad_Via, symbol Mechanical:MountingHole_Pad
- added Q1: IRFB4020, Package_TO_SOT_THT:TO-220-3_Vertical, symbol irfb4020:IRFB4020
- added SW1: SW_Push, Button_Switch_SMD:SW_Push_1P1T_NO_Vertical_Wuerth_434133025816, symbol Switch:SW_Push
- RV1: footprint Potentiometer_SMD:Potentiometer_Bourns_3269P_Horizontal -> Potentiometer_THT:Potentiometer_Bourns_3296W_Vertical
Connections:
- net CC_SET: now also U4.29 (PA8); no longer U4.30 (PA9)
- net CV_SET: now also U4.30 (PA9); no longer U4.29 (PA8)
- net ENABLE: now also U4.33 (PA12); no longer U4.26 (PB13)
- net GATE: now also Q1.1 (G)
- net GND: now also C1.2, H1.1, H2.1, H3.1, H4.1, SW1.2
- net NRST: now also C1.1, SW1.1
- net VBAT: now also Q1.2 (D)
- net VCC_SENSE: now also U4.12 (PA2); no longer U4.11 (PA1)
- net at R10.1, R9.1: now also Q1.3 (S)
- net at U4.41 (PB5): no longer D4.2 (A)
- net at U4.42 (PB6): now also D4.2 (A)

Commit message: *: Fill in info boxes
Other:
- company: (none) -> York Formula Student
- title: (none) -> Linear Battery Charger
Changed lines of the file:
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@@
 	(generator_version "9.0")
 	(paper "A4")
+	(title_block
+		(title "Linear Battery Charger")
+		(date "2025-11-22")
+		(rev "${REVISION}")
+		(company "York Formula Student")
+	)
 	(rectangle
 		(start 33.02 127)

Commit message: schematic: Switch op-amp to LM358BA
Parts:
- removed U3: OPA1678, Package_SO:SOIC-8_3.9x4.9mm_P1.27mm, symbol Amplifier_Operational:OPA1678
- added U3: LM358, Package_SO:SOIC-8_3.9x4.9mm_P1.27mm, symbol Amplifier_Operational:LM358
Connections:
- net +12V: now also U3.8 (V+)
- net CC_FB: now also U3.6 (-)
- net CV_FB: now also U3.2 (-)
- net GND: now also U3.4 (V-)
- net at C9.1, R7.1: now also U3.1
- net at C8.1, R5.2, R6.1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: now also U3.5 (+)
- net at C7.1, R2.2, TP5.1: now also U3.3 (+)
- net at C10.1, R8.1: now also U3.7

Commit message: bom: Fix incorrect 3k resistor part number
Parts:
- R14: Dist # C25804 -> C4211; Mfr # 0603WAF1002T5E -> 0603WAF3001T5E
Changed lines of the file:
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@@
 			)
 		)
-		(property "Dist #" "C25804"
+		(property "Dist #" "C4211"
 			(at 165.1 88.9 0)
 			(effects
@@
 			)
 		)
-		(property "Mfr #" "0603WAF1002T5E"
+		(property "Mfr #" "0603WAF3001T5E"
 			(at 165.1 88.9 0)
 			(effects
